Commit message: both launch scripts are working. need to add physics to the urdf. classroom world file added. the castor wobble still there. guess the issue is there in solidwork created mesh. cneters aren' aligned

File: src/robot_description/urdf/AEP_Robot.urdf (robot description, URDF)
Before this commit: robot robot_description, 8 links, 7 joints
Links:
- link base_link: mass 15.463 -> 15.896
Joints:
- joint back_castor_body_joint: limit (none) -> lower=0 upper=0 effort=0 velocity=0
- joint back_castor_wheel_joint: axis 0.056964 0.99838 0 -> 0 1 0; limit (none) -> lower=0 upper=0 effort=0 velocity=0; origin xyz=-0.023712 0.011818 -0.033 rpy=0 0 0 -> xyz=-0.024216 0.020654 -0.033 rpy=0 0 0
- joint front_castor_body_joint: limit (none) -> lower=0 upper=0 effort=0 velocity=0
- joint front_castor_wheel_joint: axis 0.10669 0.99429 0 -> 0 1 0; limit (none) -> lower=0 upper=0 effort=0 velocity=0; origin xyz=-0.02425 -0.010422 -0.033 rpy=0 0 0 -> xyz=0.021643 0.023336 -0.033 rpy=0 0 0
- joint left_wheel_joint: limit (none) -> lower=0 upper=0 effort=0 velocity=0
- joint lidar_joint: origin xyz=0 0.00042039 0.30565 rpy=0 0 0 -> xyz=0 0.000420393431200835 0.32565 rpy=0 0 0
- joint right_wheel_joint: limit (none) -> lower=0 upper=0 effort=0 velocity=0
